Commit message: demo for all except lift/drag

File: example/sailboat.xacro (robot description, xacro)
@@ -1,3 +1,3 @@
-  <?xml version="1.0" ?>
+<!-- <?xml version="1.0" ?> -->
   <!-- rigid wing with gazebo plugins for dynamics -->
   <robot name="sailboat" xmlns:xacro="http://www.ros.org/wiki/xacro">
@@ -114,5 +114,5 @@
     </link>
     <joint name="engine_propeller_joint" type="continuous">
-      <axis rpy="0 0 0" xyz="1 0 0"/>
+      <axis xyz="1 0 0"/>
       <parent link="sailboat/base_link"/>
       <child link="sailboat/propeller"/>
@@ -138,5 +138,5 @@
     <!-- Standard plugin - Thrusters and joint controllers -->
       <plugin filename="ignition-gazebo-thruster-system" name="ignition::gazebo::systems::Thruster">
-        <joint_name>sailboat/engine_propeller_joint</joint_name>
+        <joint_name>engine_propeller_joint</joint_name>
         <thrust_coefficient>0.004422</thrust_coefficient>
         <fluid_density>1000</fluid_density>
@@ -163,5 +163,5 @@
       </plugin>
     <!-- Custom plugin for simulating hull dynamics-->
-      <plugin filename="Hull" name="boating::Hull">
+      <plugin filename="boating-Hull" name="boating::Hull">
         <link_name>sailboat/base_link</link_name>
         <hull_length>6.0</hull_length>
@@ -173,5 +173,18 @@
         </points>
         <wavefield>
-          <topic>/vrx/wavefield/parameters</topic>
+          <topic>/wavefield</topic>
+        </wavefield>
+      </plugin>
+      <plugin filename="boating-Hull" name="boating::Hull">
+        <link_name>sailboat/base_link</link_name>
+        <hull_length>6.0</hull_length>
+        <hull_radius>2.5</hull_radius>
+        <fluid_level>0</fluid_level>
+        <points>
+          <point>1.4 -1.03 ${zsurf}</point>
+          <point>-1.4 -1.03 ${zsurf}</point>
+        </points>
+        <wavefield>
+          <topic>/wavefield</topic>
         </wavefield>
       </plugin>

Commit message: take in wind topic instrad of wind entity

File: example/sailboat.xacro (robot description, xacro)
@@ -2,6 +2,6 @@
   <!-- rigid wing with gazebo plugins for dynamics -->
   <robot name="sailboat" xmlns:xacro="http://www.ros.org/wiki/xacro">
-    <xacro:arg name="mast" default="0.3"/>
-    <xacro:property name="mast" value="$(arg mast)"/>
+<!--     <xacro:arg name="mast" default=""/> -->
+    <xacro:property name="mast" value="0.3"/>
     <xacro:arg name="rudder_x" default="-2.1"/>
     <xacro:arg name="rudder_z" default="-0.05"/>
@@ -218,6 +218,6 @@
       <disable_added_mass>true</disable_added_mass>
       <!-- Negative linear damping (totally random for now) -->
-      <xU>-0.1</xU>
-      <yV>-0.1</yV>
+      <xU>-10.1</xU>
+      <yV>-10.1</yV>
       <zW>-1</zW>
       <kP>-0.5</kP>

Commit message: Finished the proa boat simulation, with thrusters inside of the rudders, and rudders on the front and back of the main body. Control sliders were added as well.

File: example/sailboat.xacro (robot description, xacro)
@@ -4,6 +4,6 @@
     <xacro:arg name="mast" default="0.3"/>
     <xacro:property name="mast" value="$(arg mast)"/>
-    <xacro:arg name="rudder_x" default="-2.1"/>
-    <xacro:arg name="rudder_z" default="-0.05"/>
+    <xacro:property name="rudder_x" value="-2.1"/>
+    <xacro:property name="rudder_z" value="-0.05"/>
     <xacro:property name="zsurf" value="-0.15"/>
   <!-- Dummy inertia for now -->
@@ -28,4 +28,7 @@
       <color rgba=".3 .3 .3 1"/>
     </material>
+    <material name="red">
+      <color rgba=".9 .1 .1 1"/>
+    </material>
     <gazebo>
       <enable_wind>true</enable_wind>
@@ -58,4 +61,37 @@
       </inertial>
     </link>
+    <!--Proa Float -->
+    <link name="sailboat/proa_link">
+      <visual>
+        <geometry>
+          <mesh filename="file://$(find boating_gz)/example/mesh/hull.stl"/>
+        </geometry>
+        <material name="hull"/>
+      </visual>
+        <visual>
+        <origin xyz="0 0 ${1.5*mast}"/>
+        <geometry>
+          <cylinder length="${2*mast}" radius=".04"/>
+        </geometry>
+        <material name="grey"/>
+      </visual>
+      <!-- Simple model collision -->
+      <collision name="proa_float">
+        <geometry>
+          <mesh filename="file://$(find boating_gz)/example/mesh/hull.stl"/>
+        </geometry>
+      </collision>
+      <inertial>
+        <origin xyz="0 0 -1."/>
+        <!-- TODO update inertia -->
+        <mass value="100.0"/>
+        <inertia ixx="120.0" ixy="0.0" ixz="0.0" iyy="393" iyz="0.0" izz="446.0"/>
+      </inertial>
+    </link>
+    <joint name="proa_joint" type="fixed">
+      <parent link="sailboat/base_link"/>
+      <child link="sailboat/proa_link"/>
+      <origin rpy="0 0 0" xyz="0 -4 0"/>
+    </joint>
     <!-- wing -->
     <link name="sailboat/wing">
@@ -73,5 +109,5 @@
       <axis xyz="0 0 1"/>
       <origin rpy="0 0 0" xyz="0 0 ${2*mast}"/>
-      <limit effort="100" velocity="100" lower="${-.8*pi/2}" upper="${.8*pi/2}"/>
+      <limit effort="100" velocity="100" lower="${-pi}" upper="${pi}"/>
       <dynamics damping="0.05" friction="0.05"/>
     </joint>
@@ -90,6 +126,23 @@
       <child link="sailboat/rudder"/>
       <axis xyz="0 0 1"/>
-      <origin rpy="0 0 0" xyz="$(arg rudder_x) 0 $(arg rudder_z)"/>
-      <limit effort="100" velocity="100" lower="${-pi/4}" upper="${pi/4}"/>
+      <origin rpy="0 0 0" xyz="${rudder_x} 0 ${rudder_z}"/>
+      <limit effort="100" velocity="50" lower="${-pi}" upper="${pi}"/>
+      <dynamics damping="0.05" friction="0.05"/>
+    </joint>
+    <link name="sailboat/rudder2">
+        <visual>
+        <geometry>
+          <mesh filename="file://$(find boating_gz)/example/mesh/rudder.stl"/>
+        </geometry>
+        <material name="rudder"/>
+      </visual>
+      <xacro:inertia mass="2"/>
+    </link>
+    <joint name="rudder2_joint" type="revolute">
+      <parent link="sailboat/base_link"/>
+      <child link="sailboat/rudder2"/>
+      <axis xyz="0 0 1"/>
+      <origin rpy="0 0 0" xyz="1 0 ${rudder_z}"/>
+      <limit effort="100" velocity="50" lower="${-pi}" upper="${pi}"/>
       <dynamics damping="0.05" friction="0.05"/>
     </joint>
@@ -99,6 +152,7 @@
         <geometry>
           <mesh filename="file://$(find boating_gz)/example/mesh/propeller.dae"
-                scale=".4 .4 .4"/>
-        </geometry>
+                scale=".6 .6 .6"/>
+        </geometry>
+        <material name="red"/>
       </visual>
       <collision name="propeller_collision">
@@ -115,7 +169,34 @@
     <joint name="engine_propeller_joint" type="continuous">
       <axis xyz="1 0 0"/>
-      <parent link="sailboat/base_link"/>
+      <parent link="sailboat/rudder"/>
       <child link="sailboat/propeller"/>
-      <origin rpy="0 0 0" xyz="-1.6 0 -0.2"/>
+      <origin rpy="0 0 0" xyz="0 0 -0.2"/>
+      <limit effort="100" velocity="100"/>
+      <dynamics damping="0.05" friction="0.05"/>
+    </joint>
+    <link name="sailboat/propellerproa">
+      <visual>
+        <geometry>
+          <mesh filename="file://$(find boating_gz)/example/mesh/propeller.dae"
+                scale=".6 .6 .6"/>
+        </geometry>
+        <material name="red"/>
+      </visual>
+      <collision name="propellerproa_collision">
+        <origin rpy="0 1.57 0" xyz="-0.08 0 0"/>
+        <geometry>
+          <cylinder length="0.18" radius="0.24"/>
+        </geometry>
+      </collision>
+      <inertial>
+        <mass value="0.5"/>
+        <inertia ixx="0.008545" ixy="0.0" ixz="0.0" iyy="0.008545" iyz="0.0" izz="0.0144"/>
+      </inertial>
+    </link>
+    <joint name="engine_propellerproa_joint" type="continuous">
+      <axis xyz="1 0 0"/>
+      <parent link="sailboat/rudder2"/>
+      <child link="sailboat/propellerproa"/>
+      <origin rpy="0 0 0" xyz="0 0 -0.2"/>
       <limit effort="100" velocity="100"/>
       <dynamics damping="0.05" friction="0.05"/>
@@ -149,4 +230,16 @@
         <topic>thrust</topic>
       </plugin>
+      <plugin filename="ignition-gazebo-thruster-system" name="ignition::gazebo::systems::Thruster">
+        <joint_name>engine_propellerproa_joint</joint_name>
+        <thrust_coefficient>0.004422</thrust_coefficient>
+        <fluid_density>1000</fluid_density>
+        <propeller_diameter>0.2</propeller_diameter>
+        <velocity_control>true</velocity_control>
+        <!-- max total thrust / 2 -->
+        <max_thrust_cmd>5000.0</max_thrust_cmd>
+        <namespace>sailboat</namespace>
+        <!-- Not used by Gazebo but used to run the bridge easily -->
+        <topic>thrust2</topic>
+      </plugin>
       <plugin filename="ignition-gazebo-joint-position-controller-system" name="ignition::gazebo::systems::JointPositionController">
         <joint_name>wing_joint</joint_name>
@@ -155,9 +248,16 @@
         <name>wing</name>
       </plugin>
-        <plugin filename="ignition-gazebo-joint-position-controller-system" name="ignition::gazebo::systems::JointPositionController">
+      <plugin filename="ignition-gazebo-joint-position-controller-system" name="ignition::gazebo::systems::JointPositionController">
         <joint_name>rudder_joint</joint_name>
         <use_velocity_commands>true</use_velocity_commands>
         <!-- Not used by Gazebo but used to run the bridge easily -->
         <topic>sailboat/rudder/pos</topic>
+        <name>wing</name>
+      </plugin>
+      <plugin filename="ignition-gazebo-joint-position-controller-system" name="ignition::gazebo::systems::JointPositionController">
+        <joint_name>rudder2_joint</joint_name>
+        <use_velocity_commands>true</use_velocity_commands>
+        <!-- Not used by Gazebo but used to run the bridge easily -->
+        <topic>sailboat/rudder2/pos</topic>
         <name>wing</name>
       </plugin>
@@ -171,4 +271,6 @@
         <point>1.4 1.03 ${zsurf}</point>
         <point>-1.4 1.03 ${zsurf}</point>
+        <point>1.4 -1.03 ${zsurf}</point>
+        <point>-1.4 -1.03 ${zsurf}</point>
       </points>
       <wavefield>
@@ -176,4 +278,21 @@
       </wavefield>
     </plugin>
+    <!-- Custom plugin for simulating hull dynamics-->
+    <plugin filename="boating-Hull" name="boating::Hull">
+      <link_name>sailboat/proa_link</link_name>
+      <hull_length>6.0</hull_length>
+      <hull_radius>2.5</hull_radius>
+      <fluid_level>0</fluid_level>
+      <points>
+        <point>1.4 1.03 ${zsurf}</point>
+        <point>-1.4 1.03 ${zsurf}</point>
+        <point>1.4 -1.03 ${zsurf}</point>
+        <point>-1.4 -1.03 ${zsurf}</point>
+      </points>
+      <wavefield>
+        <topic>/wavefield</topic>
+      </wavefield>
+    </plugin>
+    <!-- Unnecessary section?
     <plugin filename="boating-Hull" name="boating::Hull">
       <link_name>sailboat/base_link</link_name>
@@ -189,7 +308,11 @@
       </wavefield>
     </plugin>
+    -->
   <!-- Standard plugin for water hydrodynamics -->
     <plugin filename="ignition-gazebo-hydrodynamics-system" name="ignition::gazebo::systems::Hydrodynamics">
       <link_name>sailboat/base_link</link_name>
+      <link_name>sailboat/proa_link</link_name>
+      <link_name>sailboat/rudder</link_name>
+      <link_name>sailboat/rudder2</link_name>
      <!-- water current topic : default to /ocean_current -->
       <!-- no added mass -->
@@ -213,4 +336,5 @@
     <plugin filename="ignition-gazebo-hydrodynamics-system" name="ignition::gazebo::systems::Hydrodynamics">
       <link_name>sailboat/base_link</link_name>
+      <link_name>sailboat/proa_link</link_name>
      <!-- air current (e.g. wind) topic: /model/wind/ocean_current
           because this plugin is designed for water current -->
@@ -218,6 +342,6 @@
       <disable_added_mass>true</disable_added_mass>
       <!-- Negative linear damping (totally random for now) -->
-      <xU>-0.1</xU>
-      <yV>-0.1</yV>
+      <xU>-1</xU>
+      <yV>-1</yV>
       <zW>-1</zW>
       <kP>-0.5</kP>
@@ -225,23 +349,38 @@
       <nR>-0.5</nR>
     </plugin>
+    <plugin
+        filename="gz-sim-lift-drag-system"
+        name="gz::sim::systems::LiftDrag">
+        <a0>0.1</a0>
+        <cla>0.1</cla>
+        <cda>0.001</cda>
+        <cma>0.0</cma>
+        <cp>0.0 0.5 0</cp>
+        <area>0.2</area>
+        <flow_topic>/model/wind/ocean_current</flow_topic>
+        <air_density>1.2041</air_density>
+        <forward>1 0 0</forward>
+        <upward>0 0 1</upward>
+        <link_name>sailboat/wing</link_name>
+      </plugin>
     <!-- Modified lift-drag plugin for wing -->
     <plugin
       filename="boating-LiftDrag"
       name="boating::LiftDrag">
-      <a0>0.2</a0>
-      <cla>10.000</cla>
+      <a0>0.087</a0>
+      <cla>5.400</cla>
       <cda>0.0001</cda>
-      <cma>0.00</cma>
-      <alpha_stall>10.0</alpha_stall>
-      <cla_stall>1.0</cla_stall>
+      <cma>0.001</cma>
+      <alpha_stall>0.33</alpha_stall>
+      <cla_stall>-2.10</cla_stall>
       <cda_stall>0.001</cda_stall>
       <cma_stall>0.0</cma_stall>
-      <cp>0.0 0.5 0</cp>
+      <cp>0.0 0 1</cp>
       <area>0.2</area>
       <!-- will guess we are in the air and subscribe to /model/wind/ocean_current -->
       <density>1.2041</density>
       <!-- to be adapted -->
-      <forward>0 0 -1</forward>
-      <upward>-1 0 0</upward>
+      <forward>-1 0 0</forward>
+      <upward>0 -1 0</upward>
       <link_name>sailboat/wing</link_name>
     </plugin>
@@ -267,4 +406,5 @@
       <upward>-1 0 0</upward>
       <link_name>sailboat/rudder</link_name>
+      <link_name>sailboat/rudder2</link_name>
     </plugin>
     </gazebo>
